Commit message: Working Baseline

File: legacy/robots/caracara_gazebo/urdf/caracara_gazebo.xacro (robot description, xacro)
@@ -15,4 +15,6 @@
   <xacro:arg name="debug" default="0"/>
   <xacro:arg name="namespace" default="caracara"/>
+  <xacro:arg name="inertial_reference_frame" default="world"/>
+  <xacro:property name="namespace" value="caracara"/>
   <!-- "Dummy" base link to eliminate root link inertia warning -->
   <link name="$(arg namespace)/base_link"/>
@@ -104,4 +106,7 @@
  <!-- Substitute the ECA A9 prop mesh for the larger uuv_descriptions one -->
  <xacro:property name="prop_mesh_file" value="file://$(find eca_a9_description)/mesh/eca_a9_propeller.dae"/>
+ <xacro:include filename="$(find uuv_sensor_ros_plugins)/urdf/camera_snippets.xacro"/>
+ <xacro:include filename="$(find uuv_sensor_ros_plugins)/urdf/sensor_snippets.xacro"/>
+ <xacro:include filename="$(find gazebo_sensors_tutorial)/robot/sensors/_d415.urdf.xacro"/>
   <!-- Thruster joint and link snippet
        Wrapper for the the thruster_module_first_order_basic_fcn_macro
@@ -114,7 +119,7 @@
   -->
   <xacro:macro name="thruster_macro"
-   	           params="thruster_id *origin">
+   	           params="namespace thruster_id *origin">
     <xacro:thruster_module_first_order_basic_fcn_macro
-        namespace="$(arg namespace)"
+        namespace="${namespace}"
         thruster_id="${thruster_id}"
         mesh_filename="${prop_mesh_file}"
@@ -125,23 +130,47 @@
   </xacro:macro>
   <!-- Port-Aft -->
-  <xacro:thruster_macro thruster_id="0">
+  <xacro:thruster_macro namespace="${namespace}" thruster_id="0">
     <origin xyz="-0.82 0.33 -0.25" rpy="${0*d2r} ${0*d2r} ${-160.0*d2r}"/>
   </xacro:thruster_macro>
   <!-- Starboard-Aft -->
-  <xacro:thruster_macro thruster_id="1">
+  <xacro:thruster_macro namespace="${namespace}" thruster_id="1">
     <origin xyz="-0.82 -0.33 -0.25" rpy="${0*d2r} ${0*d2r} ${160.0*d2r}"/>
   </xacro:thruster_macro>
   <!-- Port-Forward -->
-  <xacro:thruster_macro thruster_id="2">
+  <xacro:thruster_macro namespace="${namespace}" thruster_id="2">
     <origin xyz="0.3 0.315 -0.24" rpy="${0*d2r} ${0*d2r} ${160.0*d2r}"/>
   </xacro:thruster_macro>
   <!-- Starboard-Forward -->
-  <xacro:thruster_macro thruster_id="3">
+  <xacro:thruster_macro namespace="${namespace}" thruster_id="3">
     <origin xyz="0.3 -0.315 -0.24" rpy="${0*d2r} ${0*d2r} ${-160.0*d2r}"/>
   </xacro:thruster_macro>
   <!-- Vertical (centerline) -->
-  <xacro:thruster_macro thruster_id="4">
+  <xacro:thruster_macro namespace="${namespace}" thruster_id="4">
     <origin xyz="-0.15 0.0 0.33" rpy="${0*d2r} ${-90*d2r} ${0.0*d2r}"/>
   </xacro:thruster_macro>
+  <!-- Mount and IMU -->
+  <xacro:default_imu_macro
+    namespace="$(arg namespace)"
+    parent_link="$(arg namespace)/base_link"
+    inertial_reference_frame="$(arg inertial_reference_frame)">
+    <origin xyz="0 0 0" rpy="0 0 0"/>
+  </xacro:default_imu_macro>
+  <!-- Mount a camera -->
+  <xacro:default_camera namespace="$(arg namespace)" parent_link="$(arg namespace)/base_link" suffix="left">
+    <origin xyz=".9 0.3 0.4" rpy="0 0 0"/>
+  </xacro:default_camera>
+  <xacro:default_camera namespace="$(arg namespace)" parent_link="$(arg namespace)/base_link" suffix="right">
+    <origin xyz=".9 -0.3 0.4" rpy="0 0 0"/>
+  </xacro:default_camera>
+  <!-- Mount a RealSense -->
+  <xacro:include filename="$(find gazebo_sensors_tutorial)/robot/sensors/_d415.urdf.xacro"/>
+  <xacro:sensor_d415 name="$(arg namespace)/camera_depth" parent="$(arg namespace)/base_link" flag_color="0" flag_ir="0" flag_depth="1" updaterate="0.2">
+		<origin xyz="0.0 0 0.4" rpy="0 0 0" /> <!-- result from calib -->
+  </xacro:sensor_d415>
+  <!-- Mount a Pose 3D sensor. -->
+  <xacro:default_pose_3d_macro
+    namespace="$(arg namespace)"
+    parent_link="$(arg namespace)/base_link"
+    inertial_reference_frame="$(arg inertial_reference_frame)" />
  <!-- Default joint state publisher -->
  <gazebo>
@@ -151,3 +180,8 @@
    </plugin>
  </gazebo>
+  <include file="$(find uuv_assistants)/launch/message_to_tf.launch">
+    <arg name="namespace" value="$(arg namespace)"/>
+    <arg name="world_frame" value="world"/>
+    <arg name="child_frame_id" value="/$(arg namespace)/base_link"/>
+  </include>
 </robot>

File: urdf/robots/caracara_description/urdf/caracara.xacro (robot description, xacro)
@@ -151,3 +151,8 @@
    </plugin>
  </gazebo>
+  <include file="$(find uuv_assistants)/launch/message_to_tf.launch">
+    <arg name="namespace" value="$(arg namespace)"/>
+    <arg name="world_frame" value="world"/>
+    <arg name="child_frame_id" value="/$(arg namespace)/base_link"/>
+  </include>
 </robot>

Commit message: 9-21 update

File: legacy/robots/caracara_gazebo/urdf/caracara_gazebo.xacro (robot description, xacro)
@@ -14,10 +14,10 @@
 <robot name="caracara" xmlns:xacro="http://www.ros.org/wiki/xacro" >
   <xacro:arg name="debug" default="0"/>
-  <xacro:arg name="namespace" default="caracara"/>
+  <xacro:arg name="namespace" default="bernard"/>
   <xacro:arg name="inertial_reference_frame" default="world"/>
-  <xacro:property name="namespace" value="caracara"/>
+  <xacro:property name="namespace" value="bernard"/>
   <!-- "Dummy" base link to eliminate root link inertia warning -->
-  <link name="$(arg namespace)/base_link"/>
-  <link name="$(arg namespace)/caracara_link">
+  <!--<link name="$(arg namespace)/base_link"/>-->
+  <link name="$(arg namespace)/base_link">
     <!-- Mass and inertia from the Saab Caracara technical specifications:
          https://www.saabseaeye.com/solutions/underwater-vehicles/caracara -->
@@ -44,9 +44,9 @@
   </link>
   <!-- Attach caracara_link to the dummy base link -->
-  <joint name="$(arg namespace)/caracara_base_joint" type="fixed">
-    <origin xyz="0 0 0" rpy="0 0 0"/>  <!-- X-fwd, Y-lft, Z-up (ick!) -->
-    <parent link="$(arg namespace)/base_link"/>
+  <!--<joint name="$(arg namespace)/caracara_base_joint" type="fixed">
+    <origin xyz="0 0 0" rpy="0 0 0"/>-->  <!-- X-fwd, Y-lft, Z-up (ick!) -->
+    <!--<parent link="$(arg namespace)/base_link"/>
     <child link="$(arg namespace)/caracara_link"/>
-  </joint>
+  </joint>-->
  <gazebo>
    <plugin name="uuv_plugin" filename="libuuv_underwater_object_ros_plugin.so">
@@ -108,5 +108,5 @@
  <xacro:include filename="$(find uuv_sensor_ros_plugins)/urdf/camera_snippets.xacro"/>
  <xacro:include filename="$(find uuv_sensor_ros_plugins)/urdf/sensor_snippets.xacro"/>
- <xacro:include filename="$(find gazebo_sensors_tutorial)/robot/sensors/_d415.urdf.xacro"/>
+ <!--<xacro:include filename="$(find gazebo_sensors_tutorial)/robot/sensors/_d415.urdf.xacro"/>-->
   <!-- Thruster joint and link snippet
        Wrapper for the the thruster_module_first_order_basic_fcn_macro
@@ -153,5 +153,5 @@
     namespace="$(arg namespace)"
     parent_link="$(arg namespace)/base_link"
-    inertial_reference_frame="$(arg inertial_reference_frame)">
+    inertial_reference_frame="world">
     <origin xyz="0 0 0" rpy="0 0 0"/>
   </xacro:default_imu_macro>
@@ -164,24 +164,24 @@
   </xacro:default_camera>
   <!-- Mount a RealSense -->
-  <xacro:include filename="$(find gazebo_sensors_tutorial)/robot/sensors/_d415.urdf.xacro"/>
+  <!--<xacro:include filename="$(find gazebo_sensors_tutorial)/robot/sensors/_d415.urdf.xacro"/>
   <xacro:sensor_d415 name="$(arg namespace)/camera_depth" parent="$(arg namespace)/base_link" flag_color="0" flag_ir="0" flag_depth="1" updaterate="0.2">
-		<origin xyz="0.0 0 0.4" rpy="0 0 0" /> <!-- result from calib -->
-  </xacro:sensor_d415>
+		<origin xyz="0.0 0 0.4" rpy="0 0 0" />
+  </xacro:sensor_d415>-->
   <!-- Mount a Pose 3D sensor. -->
-  <xacro:default_pose_3d_macro
+  <!--<xacro:default_pose_3d_macro
     namespace="$(arg namespace)"
     parent_link="$(arg namespace)/base_link"
-    inertial_reference_frame="$(arg inertial_reference_frame)" />
+    inertial_reference_frame="$(arg inertial_reference_frame)" />  -->
  <!-- Default joint state publisher -->
- <gazebo>
+ <!--<gazebo>
    <plugin name="uuv_joint_state_publisher" filename="libuuv_joint_state_publisher.so">
      <robotNamespace>$(arg namespace)</robotNamespace>
      <updateRate>50</updateRate>
    </plugin>
- </gazebo>
-  <include file="$(find uuv_assistants)/launch/message_to_tf.launch">
+ </gazebo>-->
+  <!--<include file="$(find uuv_assistants)/launch/message_to_tf.launch">
     <arg name="namespace" value="$(arg namespace)"/>
     <arg name="world_frame" value="world"/>
     <arg name="child_frame_id" value="/$(arg namespace)/base_link"/>
-  </include>
+  </include>-->
 </robot>

File: urdf/dave_snippets/urdf/tasksnippets.xacro (robot description, xacro)
@@ -24,17 +24,17 @@
       <is_static>true</is_static>
     </gazebo>
-    <!--<gazebo reference="taskvisualizer/task_${number}">
+    <gazebo reference="taskvisualizer/task_${number}">
       <material value="Gazebo/${color}Glow"/>
-    </gazebo> -->
+    </gazebo>
     <joint name="taskvisualizer/task_${number}_joint" type="fixed">
       <parent link="world"/>
       <child link="taskvisualizer/task_${number}"/>
     </joint>
-    <gazebo reference='taskvisualizer/task_${number}'>
+    <!--<gazebo reference='taskvisualizer/task_${number}'>
     <visual>
       <plugin name="gazebo_ros_model_color" filename="libgazebo_ros_model_color.so">
-        <robotNamespace>/taskvisualizer/task_${number}</robotNamespace> <!-- Robot namespace -->
-        <serviceName>/task${number}_color</serviceName> <!-- Service topic name-->
-        <color>1.0 1.0 1.0 1.0</color> <!-- Default Color -->
+        <robotNamespace>/taskvisualizer/task_${number}</robotNamespace>
+        <serviceName>/task${number}_color</serviceName>
+        <color>1.0 1.0 1.0 1.0</color>
       </plugin>
     </visual>
@@ -44,5 +44,5 @@
       <robotNamespace>/taskvisualizer/task_${number}</robotNamespace>
     </plugin>
-  </gazebo>
+  </gazebo>-->
   </xacro:macro>
 </robot>

File: urdf/dave_snippets/urdf/ui_gazebo.xacro (robot description, xacro)
@@ -22,12 +22,12 @@
   </gazebo>
   <link name="world"/>
-  <!-- Options for color are: Red, Blue, Yellow, Green, White, Purple, Turquoise. Gazebo stores materials at
+  <!-- Options for color are: Red, Blue, Yellow, Green, White, Purple(more of a pink really), Turquoise (cyan). Gazebo stores materials at
   /usr/share/gazebo-11/media/materials/scripts/gazebo.material -->
   <xacro:task_vis
-    x="0"
+    x="-5"
     y="-8"
     z="-17"
-    color="White"
-    number="1">
+    color="Blue"
+    number="11">
   </xacro:task_vis>
   <xacro:task_vis
@@ -35,27 +35,27 @@
     y="-8"
     z="-17"
-    color="White"
-    number="2">
+    color="Blue"
+    number="12">
   </xacro:task_vis>
   <xacro:task_vis
-    x="15"
+    x="-25"
     y="-8"
     z="-17"
-    color="White"
-    number="3">
+    color="Blue"
+    number="13">
   </xacro:task_vis>
   <xacro:task_vis
-    x="0"
+    x="-10"
     y="-13"
     z="-30"
-    color="White"
-    number="4">
+    color="Turquoise"
+    number="21">
   </xacro:task_vis>
   <xacro:task_vis
-    x="20.5"
+    x="-30"
     y="-13"
     z="-30"
-    color="White"
-    number="5">
+    color="Turquoise"
+    number="22">
   </xacro:task_vis>
   <xacro:task_vis
@@ -63,27 +63,27 @@
     y="-13"
     z="-30"
-    color="White"
-    number="6">
+    color="Turquoise"
+    number="23">
   </xacro:task_vis>
   <xacro:task_vis
-    x="0"
-    y="-8"
-    z="-44"
-    color="White"
-    number="7">
+    x="-8"
+    y="-12"
+    z="-23"
+    color="Yellow"
+    number="31">
   </xacro:task_vis>
   <xacro:task_vis
     x="-15"
-    y="-8"
-    z="-44"
-    color="White"
-    number="8">
+    y="-12"
+    z="-23"
+    color="Yellow"
+    number="32">
   </xacro:task_vis>
   <xacro:task_vis
-    x="15"
-    y="-8"
-    z="-44"
-    color="White"
-    number="9">
+    x="-22"
+    y="-12"
+    z="-23"
+    color="Yellow"
+    number="33">
   </xacro:task_vis>
 </robot>
